Commit message: add ur10-gripper model

File: ur10-gripper.urdf (robot description, URDF)
Before this commit: robot robotiq-3f-gripper_articulated, 13 links, 12 joints
Links:
- added link base_link, mass 4.0; collision mesh filename=meshes/ur10/collision/Base.dae; visual mesh filename=meshes/ur10/visual/Base.dae
- added link forearm_link, mass 3.87; collision mesh filename=meshes/ur10/collision/Forearm.dae; visual mesh filename=meshes/ur10/visual/Forearm.dae
- added link shoulder_link, mass 7.778; collision mesh filename=meshes/ur10/collision/Shoulder.dae; visual mesh filename=meshes/ur10/visual/Shoulder.dae
- added link upper_arm_link, mass 12.93; collision mesh filename=meshes/ur10/collision/UpperArm.dae; visual mesh filename=meshes/ur10/visual/UpperArm.dae
- added link world
- added link wrist_1_link, mass 1.96; collision mesh filename=meshes/ur10/collision/Wrist1.dae; visual mesh filename=meshes/ur10/visual/Wrist1.dae
- added link wrist_2_link, mass 1.96; collision mesh filename=meshes/ur10/collision/Wrist2.dae; visual mesh filename=meshes/ur10/visual/Wrist2.dae
- added link wrist_3_link, mass 0.202; collision mesh filename=meshes/ur10/collision/Wrist3.dae; visual mesh filename=meshes/ur10/visual/Wrist3.dae
Joints:
- added joint ee_fixed_joint: type fixed, parent wrist_3_link, child palm, origin xyz=0 0.147 0 rpy=0 0 0
- added joint elbow_joint: type revolute, parent upper_arm_link, child forearm_link, origin xyz=0.0 -0.1719 0.612 rpy=0.0 0.0 0.0, axis 0 1 0, limit lower=-6.2831853 upper=6.2831853 effort=150.0 velocity=3.15
- added joint shoulder_lift_joint: type revolute, parent shoulder_link, child upper_arm_link, origin xyz=0.0 0.220941 0.0 rpy=0.0 1.570796325 0.0, axis 0 1 0, limit lower=-6.2831853 upper=6.2831853 effort=330.0 velocity=2.16
- added joint shoulder_pan_joint: type revolute, parent base_link, child shoulder_link, origin xyz=0.0 0.0 0.1273 rpy=0.0 0.0 0.0, axis 0 0 1, limit lower=-6.2831853 upper=6.2831853 effort=330.0 velocity=2.16
- added joint world_joint: type fixed, parent world, child base_link, origin xyz=0.0 0.0 0.0 rpy=0.0 0.0 0.0
- added joint wrist_1_joint: type revolute, parent forearm_link, child wrist_1_link, origin xyz=0.0 0.0 0.5723 rpy=0.0 1.570796325 0.0, axis 0 1 0, limit lower=-6.2831853 upper=6.2831853 effort=54.0 velocity=3.2
- added joint wrist_2_joint: type revolute, parent wrist_1_link, child wrist_2_link, origin xyz=0.0 0.1149 0.0 rpy=0.0 0.0 0.0, axis 0 0 1, limit lower=-6.2831853 upper=6.2831853 effort=54.0 velocity=3.2
- added joint wrist_3_joint: type revolute, parent wrist_2_link, child wrist_3_link, origin xyz=0.0 0.0 0.1157 rpy=0.0 0.0 0.0, axis 0 1 0, limit lower=-6.2831853 upper=6.2831853 effort=54.0 velocity=3.2
