Commit message: add ur5-gripper simulator

File: ur5e-gripper.urdf (robot description, URDF)
Before this commit: robot ur10, 21 links, 20 joints
Links:
- added link base
- added link ee_link; collision box size=0.01 0.01 0.01; visual box size=0.01 0.01 0.01
- added link tool0
- link base_link: geometry collision mesh filename=./meshes/ur5e/collision/base.stl scale=1.0 1.0 1.0; visual mesh filename=./meshes/ur5e/visual/base.dae
- link forearm_link: mass 3.87 -> 2.275; geometry collision mesh filename=./meshes/ur5e/collision/forearm.stl scale=1.0 1.0 1.0; visual mesh filename=./meshes/ur5e/visual/forearm.dae
- link shoulder_link: mass 7.778 -> 3.7; geometry collision mesh filename=./meshes/ur5e/collision/shoulder.stl scale=1.0 1.0 1.0; visual mesh filename=./meshes/ur5e/visual/shoulder.dae
- link upper_arm_link: mass 12.93 -> 8.393; geometry collision mesh filename=./meshes/ur5e/collision/upperarm.stl scale=1.0 1.0 1.0; visual mesh filename=./meshes/ur5e/visual/upperarm.dae
- link wrist_1_link: mass 1.96 -> 1.219; geometry collision mesh filename=./meshes/ur5e/collision/wrist1.stl scale=1.0 1.0 1.0; visual mesh filename=./meshes/ur5e/visual/wrist1.dae
- link wrist_2_link: mass 1.96 -> 1.219; geometry collision mesh filename=./meshes/ur5e/collision/wrist2.stl scale=1.0 1.0 1.0; visual mesh filename=./meshes/ur5e/visual/wrist2.dae
- link wrist_3_link: mass 0.202 -> 0.1879; geometry collision mesh filename=./meshes/ur5e/collision/wrist3.stl scale=1.0 1.0 1.0; visual mesh filename=./meshes/ur5e/visual/wrist3.dae
Joints:
- added joint base_link-base_fixed_joint: type fixed, parent base_link, child base, origin xyz=0 0 0 rpy=0 0 -3.14159265359
- added joint ee_link_palm_joint: type fixed, parent ee_link, child palm, origin xyz=0.047 0 0 rpy=0 0 -1.5708, axis 0 0 0, limit lower=-6.2831853 upper=6.2831853 effort=100 velocity=100
- added joint wrist_3_link-tool0_fixed_joint: type fixed, parent wrist_3_link, child tool0, origin xyz=0 0.1 0 rpy=-1.57079632679 0 0
- joint ee_fixed_joint: child palm -> ee_link; origin xyz=0 0.147 0 rpy=0 0 0 -> xyz=0.0 0.1 0.0 rpy=0.0 0.0 1.57079632679
- joint elbow_joint: limit lower=-6.2831853 upper=6.2831853 effort=150.0 velocity=3.15 -> lower=-3.14159265359 upper=3.14159265359 effort=150.0 velocity=3.14; origin xyz=0.0 -0.1719 0.612 rpy=0.0 0.0 0.0 -> xyz=0.0 -0.131 0.425 rpy=0.0 0.0 0.0
- joint shoulder_lift_joint: limit lower=-6.2831853 upper=6.2831853 effort=330.0 velocity=2.16 -> lower=-6.28318530718 upper=6.28318530718 effort=150.0 velocity=3.14; origin xyz=0.0 0.220941 0.0 rpy=0.0 1.570796325 0.0 -> xyz=0.0 0.138 0.0 rpy=0.0 1.57079632679 0.0
- joint shoulder_pan_joint: limit lower=-6.2831853 upper=6.2831853 effort=330.0 velocity=2.16 -> lower=-6.28318530718 upper=6.28318530718 effort=150.0 velocity=3.14; origin xyz=0.0 0.0 0.1273 rpy=0.0 0.0 0.0 -> xyz=0.0 0.0 0.163 rpy=0.0 0.0 0.0
- joint wrist_1_joint: limit lower=-6.2831853 upper=6.2831853 effort=54.0 velocity=3.2 -> lower=-6.28318530718 upper=6.28318530718 effort=28.0 velocity=6.28; origin xyz=0.0 0.0 0.5723 rpy=0.0 1.570796325 0.0 -> xyz=0.0 0.0 0.392 rpy=0.0 1.57079632679 0.0
- joint wrist_2_joint: limit lower=-6.2831853 upper=6.2831853 effort=54.0 velocity=3.2 -> lower=-6.28318530718 upper=6.28318530718 effort=28.0 velocity=6.28; origin xyz=0.0 0.1149 0.0 rpy=0.0 0.0 0.0 -> xyz=0.0 0.127 0.0 rpy=0.0 0.0 0.0
- joint wrist_3_joint: limit lower=-6.2831853 upper=6.2831853 effort=54.0 velocity=3.2 -> lower=-6.28318530718 upper=6.28318530718 effort=28.0 velocity=6.28; origin xyz=0.0 0.0 0.1157 rpy=0.0 0.0 0.0 -> xyz=0.0 0.0 0.1 rpy=0.0 0.0 0.0
